File: Hardware/supercon-2019-blink/supercon-2019-blink.sch (KiCad schematic (older format))
At the start: 17 parts, among them J1 Conn_01x06, U1 ATtiny84A-SSU, X1 Badgelife_sao_connector_v169b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

Commit message: Gunter art layers done!
Parts:
- X1: footprint badgelife_sao_v169bis:Badgelife-SAOv169-SAO-2x3 -> footprints:Badgelife-SAOv169-SAO-2x3_nopin1
Changed lines of the file:
@@
 F 0 "X1" V 5435 5550 50  0000 C CNN
 F 1 "Badgelife_sao_connector_v169bis" V 5526 5550 50  0000 C CNN
-F 2 "badgelife_sao_v169bis:Badgelife-SAOv169-SAO-2x3" H 5900 5750 50  0001 C CNN
+F 2 "footprints:Badgelife-SAOv169-SAO-2x3_nopin1" H 5900 5750 50  0001 C CNN
 F 3 "" H 5900 5750 50  0001 C CNN
 F 4 "732-5394-ND" V 5900 5550 50  0001 C CNN "Digi-Key_PN"
