File: Hardware/supercon-2019-blink/supercon-2019-blink.kicad_pcb (KiCad board)
At the start: 2 copper layers, 43.1 x 63.6 mm, 17 parts, among them J1 Conn_01x06, U1 ATtiny84A-SSU, X1 Badgelife_sao_connector_v169b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

Commit message: Gunter art layers done!
Parts:
- added G***: LOGO, footprints:gunter-silk, F.Cu at (148.6, 95.2)
- added G***: LOGO, footprints:gunter-exposed_copper, F.Cu at (139.7, 79.5)
- added G***: LOGO, footprints:gunter-sm_keepout, F.Cu at (139.7, 79.5)
- added G***: LOGO, footprints:gunter-outer, F.Cu at (148.6, 95.0)
- X1: footprint badgelife_sao_v169bis:Badgelife-SAOv169-SAO-2x3 -> footprints:Badgelife-SAOv169-SAO-2x3_nopin1
- moved C1 7.87 mm to (156.2, 86.4)
- moved R1 7.62 mm to (153.7, 86.4)
- moved R8 6.60 mm to (151.1, 86.4)
- moved R3 6.12 mm to (144.8, 101.6), turned to 90 degrees
- moved R9 4.83 mm to (148.6, 86.4)
- moved R7 4.06 mm to (146.1, 86.4)
- moved JP1 2.68 mm to (143.5, 105.4), turned to 0 degrees
- moved R4 2.29 mm to (138.4, 86.4)
- moved J1 2.18 mm to (158.8, 99.1)
- moved D2 1.85 mm to (147.3, 78.7)
- moved R2 1.80 mm to (142.2, 101.6), turned to 90 degrees
- moved R6 1.52 mm to (141.0, 86.4)
- moved D1 0.81 mm to (134.7, 78.7), turned to 0 degrees
- moved C2 0.57 mm to (137.2, 95.2)
- moved R5 0.51 mm to (143.5, 86.4)
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
Commit message: v01 PCB layout complete
Parts:
- added G***: LOGO, footprints:gunter-back_silk, B.Cu at (148.6, 95.2)
- added G***: LOGO, footprints:DigiKey-Logo_12x6mm_SilkScreen, B.Cu at (162.4, 112.3)
- added G***: LOGO, footprints:Shawn-Logo_6x6mm_SilkScreen, B.Cu at (137.0, 112.3)
- added REF**: led_sm_keepout, footprints:led_sm_keepout, B.Cu at (134.7, 78.7)
- added REF**: led_sm_keepout, footprints:led_sm_keepout, B.Cu at (147.3, 78.7)
- added REF**: KiCad-Logo2_5mm_SilkScreen, Symbol:KiCad-Logo2_5mm_SilkScreen, B.Cu at (148.7, 112.3)
- moved JP1 1.27 mm to (143.5, 106.7)
- moved R2 1.27 mm to (142.2, 102.9)
- moved R3 1.27 mm to (144.8, 102.9)
- turned C1 to 90 degrees
Routing:
- net VCC: track 0.00 -> 109.9 mm
- net GND: track 0.00 -> 80.4 mm, vias 0 -> 7
- net MOSI_SDA: track 0.00 -> 54.5 mm, vias 0 -> 2
- net SCK_SCL: track 0.00 -> 51.0 mm, vias 0 -> 2
- net RST: track 0.00 -> 28.5 mm, vias 0 -> 2
- net Net-(D1-Pad3): track 0.00 -> 19.4 mm
- net LED_B_BLUE: track 0.00 -> 16.9 mm, vias 0 -> 2
- net LED_B_GREEN: track 0.00 -> 16.4 mm, vias 0 -> 2
- net MISO: track 0.00 -> 12.9 mm, vias 0 -> 2
- net LED_A_RED: track 0.00 -> 11.4 mm, vias 0 -> 2
- net Net-(D1-Pad4): track 0.00 -> 10.6 mm
- net Net-(D2-Pad1): track 0.00 -> 10.3 mm
- net Net-(D2-Pad4): track 0.00 -> 8.31 mm
- net Net-(D2-Pad3): track 0.00 -> 6.61 mm
- net Net-(D1-Pad1): track 0.00 -> 6.56 mm
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- added copper zone on B.Cu, net GND
Other:
- net class Default: clearance 0.2 -> 0.254; trace_width 0.25 -> 0.254; via_dia 0.8 -> 0.9144; via_drill 0.4 -> 0.4064
- rule trace_clearance: 0.2 -> 0.254
- rule trace_min: 0.2 -> 0.1524
- rule via_min_drill: 0.3 -> 0.3302
- rule via_min_size: 0.4 -> 0.6858
- board text added: "v01"

Commit message: Added silk labels to ISP header
Routing:
- net GND: track 80.4 -> 79.4 mm
- net MISO: track 12.9 -> 12.3 mm
Other:
- board text added: "GND"
- board text added: "MISO"
- board text added: "MOSI"
- board text added: "RST"
- board text added: "SCK"
- board text added: "VCC"
Changed lines of the file:
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@@
   (general
     (thickness 1.6)
-    (drawings 49)
-    (tracks 180)
+    (drawings 55)
+    (tracks 181)
     (zones 0)
     (modules 27)
@@
   )
   (layers
-    (0 F.Cu signal hide)
-    (31 B.Cu signal hide)
+    (0 F.Cu signal)
+    (31 B.Cu signal)
     (32 B.Adhes user)
     (33 F.Adhes user)
@@
     (35 F.Paste user)
     (36 B.SilkS user)
-    (37 F.SilkS user hide)
+    (37 F.SilkS user)
     (38 B.Mask user)
     (39 F.Mask user hide)
@@
   )
   (setup
-    (last_trace_width 0.254)
+    (last_trace_width 0.508)
     (user_trace_width 0.508)
     (trace_clearance 0.254)
@@
     )
   )
+  (gr_text MISO (at 151.638 105.41) (layer B.SilkS)
+    (effects (font (size 1 1) (thickness 0.15)) (justify left mirror))
+  )
+  (gr_text VCC (at 151.765 102.87) (layer B.SilkS)
+    (effects (font (size 1 1) (thickness 0.15)) (justify left mirror))
+  )
+  (gr_text SCK (at 151.765 100.33) (layer B.SilkS)
+    (effects (font (size 1 1) (thickness 0.15)) (justify left mirror))
+  )
+  (gr_text MOSI (at 151.765 97.79) (layer B.SilkS)
+    (effects (font (size 1 1) (thickness 0.15)) (justify left mirror))
+  )
+  (gr_text RST (at 151.765 95.25) (layer B.SilkS)
+    (effects (font (size 1 1) (thickness 0.15)) (justify left mirror))
+  )
+  (gr_text GND (at 151.765 92.71) (layer B.SilkS)
+    (effects (font (size 1 1) (thickness 0.15)) (justify left mirror))
+  )
   (gr_text v01 (at 166.37 122.428 45) (layer B.Cu)
     (effects (font (size 1.5 1.5) (thickness 0.3)) (justify mirror))
@@
   (segment (start 147.7864 122.956) (end 139.7 114.8696) (width 0.508) (layer B.Cu) (net 2))
   (segment (start 149.158 122.956) (end 147.7864 122.956) (width 0.508) (layer B.Cu) (net 2))
-  (via (at 150.368 92.71) (size 0.9144) (drill 0.4064) (layers F.Cu B.Cu) (net 2))
-  (segment (start 150.368 90.17) (end 150.368 92.71) (width 0.508) (layer F.Cu) (net 2))
-  (segment (start 146.05 90.795962) (end 146.05 90.126446) (width 0.508) (layer F.Cu) (net 2))
-  (segment (start 146.05 90.126446) (end 147.022446 89.154) (width 0.508) (layer F.Cu) (net 2))
-  (segment (start 147.022446 89.154) (end 149.352 89.154) (width 0.508) (layer F.Cu) (net 2))
-  (segment (start 149.352 89.154) (end 150.368 90.17) (width 0.508) (layer F.Cu) (net 2))
   (via (at 138.43 90.424) (size 0.9144) (drill 0.4064) (layers F.Cu B.Cu) (net 2))
   (segment (start 139.7 97.145962) (end 139.7 99.568) (width 0.508) (layer F.Cu) (net 2))
   (segment (start 138.43 95.875962) (end 139.7 97.145962) (width 0.508) (layer F.Cu) (net 2))
-  (segment (start 144.135962 92.71) (end 146.05 90.795962) (width 0.508) (layer F.Cu) (net 2))
-  (segment (start 138.43 92.71) (end 144.135962 92.71) (width 0.508) (layer F.Cu) (net 2))
   (segment (start 138.43 90.424) (end 138.43 92.71) (width 0.508) (layer F.Cu) (net 2))
   (via (at 153.924 83.566) (size 0.9144) (drill 0.4064) (layers F.Cu B.Cu) (net 2))
@@
   (segment (start 138.43 94.234) (end 138.43 95.875962) (width 0.508) (layer F.Cu) (net 2))
   (segment (start 138.43 92.71) (end 138.43 94.234) (width 0.508) (layer F.Cu) (net 2))
+  (via (at 150.368 91.694) (size 0.9144) (drill 0.4064) (layers F.Cu B.Cu) (net 2))
+  (segment (start 146.05 90.795962) (end 146.05 90.126446) (width 0.508) (layer F.Cu) (net 2))
+  (segment (start 138.43 92.71) (end 144.135962 92.71) (width 0.508) (layer F.Cu) (net 2))
+  (segment (start 149.352 89.154) (end 150.368 90.17) (width 0.508) (layer F.Cu) (net 2))
+  (segment (start 147.022446 89.154) (end 149.352 89.154) (width 0.508) (layer F.Cu) (net 2))
+  (segment (start 146.05 90.126446) (end 147.022446 89.154) (width 0.508) (layer F.Cu) (net 2))
+  (segment (start 144.135962 92.71) (end 146.05 90.795962) (width 0.508) (layer F.Cu) (net 2))
+  (segment (start 150.368 90.17) (end 150.368 91.694) (width 0.508) (layer F.Cu) (net 2))
   (segment (start 137.347 78.015) (end 139.991 78.015) (width 0.254) (layer B.Cu) (net 3))
   (segment (start 139.991 78.015) (end 140.97 78.994) (width 0.254) (layer B.Cu) (net 3))
@@
   (via (at 147.32 99.568) (size 0.9144) (drill 0.4064) (layers F.Cu B.Cu) (net 9))
   (segment (start 147.32 97.696) (end 147.32 99.568) (width 0.254) (layer B.Cu) (net 9))
-  (via (at 148.59 105.41) (size 0.9144) (drill 0.4064) (layers F.Cu B.Cu) (net 9))
-  (segment (start 147.32 99.568) (end 147.32 104.14) (width 0.254) (layer F.Cu) (net 9))
-  (segment (start 147.32 104.14) (end 148.59 105.41) (width 0.254) (layer F.Cu) (net 9))
-  (segment (start 148.59 105.41) (end 153.225 105.41) (width 0.254) (layer B.Cu) (net 9))
+  (via (at 148.717 104.521) (size 0.9144) (drill 0.4064) (layers F.Cu B.Cu) (net 9))
+  (segment (start 149.606 105.41) (end 148.717 104.521) (width 0.254) (layer B.Cu) (net 9))
+  (segment (start 153.225 105.41) (end 149.606 105.41) (width 0.254) (layer B.Cu) (net 9))
+  (segment (start 147.32 103.124) (end 148.717 104.521) (width 0.254) (layer F.Cu) (net 9))
+  (segment (start 147.32 99.568) (end 147.32 103.124) (width 0.254) (layer F.Cu) (net 9))
   (via (at 138.43 111.76) (size 0.9144) (drill 0.4064) (layers F.Cu B.Cu) (net 10))
   (via (at 146.05 99.568) (size 0.9144) (drill 0.4064) (layers F.Cu B.Cu) (net 10))
@@
   (segment (start 155.702 88.9) (end 157.734 90.932) (width 0.254) (layer B.Cu) (net 12))
   (segment (start 153.67 88.392) (end 153.67 88.9) (width 0.254) (layer B.Cu) (net 12))
-  (segment (start 152.908 88.138) (end 153.67 88.9) (width 0.254) (layer F.Cu) (net 12))
   (segment (start 143.51 90.424) (end 145.796 88.138) (width 0.254) (layer F.Cu) (net 12))
   (segment (start 145.796 88.138) (end 152.908 88.138) (width 0.254) (layer F.Cu) (net 12))
+  (segment (start 152.908 88.138) (end 153.67 88.9) (width 0.254) (layer F.Cu) (net 12))
   (segment (start 144.78 106.65) (end 144.81 106.68) (width 0.254) (layer B.Cu) (net 13))
   (segment (start 144.78 103.6575) (end 144.78 106.65) (width 0.254) (layer B.Cu) (net 13))
