File: Hardware/wenk_sao/wenk_sao.sch (KiCad schematic (older format))
At the start: 17 parts, among them J1 Conn_01x06, U1 ATtiny84A-SSU, X1 Badgelife_sao_connector_v169b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

Commit message: Added exercises and python uploader script
Parts:
- D1, D2: symbol XZMDKCBDDG45S-9:LED_RABG -> wenk_sao-rescue:LED_RABG-XZMDKCBDDG45S-9
- X1: symbol badgelife_shitty_addon_v169bis:Badgelife_sao_connector_v169bis -> wenk_sao-rescue:Badgelife_sao_connector_v169bis-badgelife_shitty_addon_v169bis
Other:
- moved on the sheet: C1, C2, D1, D2, J1, JP1, R1, R2, R3, R4, R5, R6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
